Commit message: add link

File: project/drive/urdf/robot_description.xacro (robot description, xacro)
@@ -2,4 +2,22 @@
 <robot name="mock_robot" xmlns:xacro="http://www.ros.org/wiki/xacro">
   <!-- The robot link description -->
-  <link name="base_link" />
+  <link name="base_link">
+    <visual>
+      <geometry>
+        <cylinder length="0.6" radius="0.2"/>
+      </geometry>
+      <material name="blue">
+        <color rgba="0 0 .8 1"/>
+      </material>
+    </visual>
+    <collision>
+      <geometry>
+        <cylinder length="0.6" radius="0.2"/>
+      </geometry>
+    </collision>
+    <inertial>
+      <mass value="10"/>
+      <inertia ixx="0.4" ixy="0.0" ixz="0.0" iyy="0.4" iyz="0.0" izz="0.2"/>
+    </inertial>
+  </link>
 </robot>
